File: Overview Sheet/Overview Sheet.kicad_pcb (KiCad board)
At the start: 4 copper layers, 129.5 x 116.5 mm, 16 parts

Commit message: Updated Links
Other:
- board text added: "Finns Constrains https://github.com/fibergm/Default-Fullstack-Project"
- board text removed: "Finns Constrains https://github.com/fibergm/KiCad-Default-Project"
Changed lines of the file:
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@@
 		)
 	)
-	(gr_text "Finns Constrains \nhttps://github.com/fibergm/KiCad-Default-Project"
+	(gr_text "Finns Constrains \nhttps://github.com/fibergm/Default-Fullstack-Project"
 		(at 61.1 22.1 0)
 		(layer "User.1")
